File: pcb/vapelight.kicad_pcb (KiCad board)
At the start: 2 copper layers, 58.2 x 15 mm, 46 parts, among them J1 USB_A, J2 Conn_01x01_Socket, J3 Conn_01x01_Socket, J4 Conn_01x01_Socket, J5 Conn_01x01_Socket, Q1 FS8205A, SW1 SW_Push, U1 DW01A, U2 LTC4054ES5-4.2, U3 LM27313XMF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

Commit message: Revision F
– less bright charge LED
– higher button
– different sizes of panelized fabrication outputs
- minor fixes
Parts:
- R1: value 180 -> 1k
Other:
- board text added: "Rev.${REVISION} ${ISSUE_DATE} CERN OHL P 2.0 https:// github.com/ sbyd-space/ vape-light"
- board text removed: "Rev.E 03/2025 CERN OHL P 2.0 https:// github.com/ sbyd-space/ vape-light"
Changed lines of the file:
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@@
 	(title_block
 		(title "vapelight")
-		(date "2025-03-05")
-		(rev "E")
+		(date "05/2025")
+		(rev "F")
 		(company "SBYD")
 	)
@@
 		(property ki_fp_filters "SOT?23* Texas?R-PDSO-G5?DCK* Texas?R-PDSO-N5?DRL* Texas?X2SON*0.8x0.8mm*P0.48mm*")
 		(sheetname "Root")
-		(sheetfile "SBYD_vape.kicad_sch")
+		(sheetfile "vapelight.kicad_sch")
 		(attr smd)
 		(fp_line
@@
 		(property ki_fp_filters "R_*")
 		(sheetname "Root")
-		(sheetfile "SBYD_vape.kicad_sch")
+		(sheetfile "vapelight.kicad_sch")
 		(attr smd)
 		(fp_line
@@
 		(property ki_fp_filters "R_*")
 		(sheetname "Root")
-		(sheetfile "SBYD_vape.kicad_sch")
+		(sheetfile "vapelight.kicad_sch")
 		(attr smd)
 		(fp_line
@@
 			)
 		)
+		(property ki_fp_filters "SolderJumper*Bridged123*")
+		(sheetname "Root")
+		(sheetfile "vapelight.kicad_sch")
 		(zone_connect 1)
 		(attr exclude_from_pos_files exclude_from_bom)
@@
 		(property ki_fp_filters "Connector*:*_1x??_*")
 		(sheetname "Root")
-		(sheetfile "SBYD_vape.kicad_sch")
+		(sheetfile "vapelight.kicad_sch")
 		(attr through_hole exclude_from_pos_files exclude_from_bom)
 		(fp_circle
@@
 		(property ki_fp_filters "R_*")
 		(sheetname "Root")
-		(sheetfile "SBYD_vape.kicad_sch")
+		(sheetfile "vapelight.kicad_sch")
 		(attr smd)
 		(fp_line
@@
 		(property ki_fp_filters "LED* LED_SMD:* LED_THT:*")
 		(sheetname "Root")
-		(sheetfile "SBYD_vape.kicad_sch")
+		(sheetfile "vapelight.kicad_sch")
 		(attr smd)
 		(fp_line
@@
 		(property ki_fp_filters "Connector*:*_1x??_*")
 		(sheetname "Root")
-		(sheetfile "SBYD_vape.kicad_sch")
+		(sheetfile "vapelight.kicad_sch")
 		(attr through_hole exclude_from_pos_files exclude_from_bom)
 		(fp_circle
@@
 			)
 		)
-		(attr exclude_from_pos_files exclude_from_bom)
+		(attr board_only exclude_from_pos_files exclude_from_bom dnp)
 		(fp_line
 			(start 0.25 0)
@@
 		(property ki_fp_filters "TSOT?23*")
 		(sheetname "Root")
-		(sheetfile "SBYD_vape.kicad_sch")
+		(sheetfile "vapelight.kicad_sch")
 		(attr smd)
 		(fp_line
@@
 			)
 		)
-		(attr exclude_from_pos_files exclude_from_bom)
+		(attr board_only exclude_from_pos_files exclude_from_bom dnp)
 		(fp_line
 			(start 0.25 1)
@@
 		(property ki_fp_filters "C_*")
 		(sheetname "Root")
-		(sheetfile "SBYD_vape.kicad_sch")
+		(sheetfile "vapelight.kicad_sch")
 		(attr smd)
 		(fp_line
@@
 		(property ki_fp_filters "R_*")
 		(sheetname "Root")
-		(sheetfile "SBYD_vape.kicad_sch")
+		(sheetfile "vapelight.kicad_sch")
 		(attr smd)
 		(fp_line
@@
 			)
 		)
-		(attr exclude_from_pos_files exclude_from_bom)
+		(attr board_only exclude_from_pos_files exclude_from_bom dnp)
 		(fp_line
 			(start 0.25 0)
@@
 			)
 		)
+		(property ki_fp_filters "SolderJumper*Bridged12*")
+		(sheetname "Root")
+		(sheetfile "vapelight.kicad_sch")
 		(zone_connect 1)
 		(attr exclude_from_pos_files exclude_from_bom)
@@
 		(property ki_fp_filters "R_*")
 		(sheetname "Root")
-		(sheetfile "SBYD_vape.kicad_sch")
+		(sheetfile "vapelight.kicad_sch")
 		(attr smd)
 		(fp_line
@@
 		(property ki_fp_filters "Connector*:*_1x??_*")
 		(sheetname "Root")
-		(sheetfile "SBYD_vape.kicad_sch")
+		(sheetfile "vapelight.kicad_sch")
 		(attr through_hole exclude_from_pos_files exclude_from_bom)
 		(fp_circle
@@
 		(property ki_fp_filters "R_*")
 		(sheetname "Root")
-		(sheetfile "SBYD_vape.kicad_sch")
+		(sheetfile "vapelight.kicad_sch")
 		(attr smd)
 		(fp_line
@@
 		(property ki_fp_filters "Connector*:*_1x??_*")
 		(sheetname "Root")
-		(sheetfile "SBYD_vape.kicad_sch")
+		(sheetfile "vapelight.kicad_sch")
 		(attr through_hole exclude_from_pos_files exclude_from_bom)
 		(fp_circle
@@
 		(property ki_fp_filters "TO-???* *_Diode_* *SingleDiode* D_*")
 		(sheetname "Root")
-		(sheetfile "SBYD_vape.kicad_sch")
+		(sheetfile "vapelight.kicad_sch")
 		(attr smd)
 		(fp_line
@@
 		)
 		(sheetname "Root")
-		(sheetfile "SBYD_vape.kicad_sch")
+		(sheetfile "vapelight.kicad_sch")
 		(attr smd)
 		(fp_line
@@
 			)
 		)
-		(property "Value" "180"
+		(property "Value" "1k"
 			(at 0 1.43 -90)
 			(layer "F.Fab")
@@
 			)
 		)
-		(property "LCSC" "C22828"
+		(property "LCSC" "C21190"
 			(at 0 0 90)
 			(unlocked yes)
@@
 		(property ki_fp_filters "R_*")
 		(sheetname "Root")
-		(sheetfile "SBYD_vape.kicad_sch")
+		(sheetfile "vapelight.kicad_sch")
 		(attr smd)
 		(fp_line
@@
 		(property ki_fp_filters "SOT* SC*")
 		(sheetname "Root")
-		(sheetfile "SBYD_vape.kicad_sch")
+		(sheetfile "vapelight.kicad_sch")
 		(attr smd)
 		(fp_line
@@
 			)
 		)
-		(attr exclude_from_pos_files exclude_from_bom)
+		(attr board_only exclude_from_pos_files exclude_from_bom dnp)
 		(fp_line
 			(start 0.25 1)
@@
 		(property ki_fp_filters "C_*")
 		(sheetname "Root")
-		(sheetfile "SBYD_vape.kicad_sch")
+		(sheetfile "vapelight.kicad_sch")
 		(attr smd)
 		(fp_line
@@
 		(property ki_fp_filters "C_*")
 		(sheetname "Root")
-		(sheetfile "SBYD_vape.kicad_sch")
+		(sheetfile "vapelight.kicad_sch")
 		(attr smd)
 		(fp_line
@@
 		(property ki_fp_filters "R_*")
 		(sheetname "Root")
-		(sheetfile "SBYD_vape.kicad_sch")
+		(sheetfile "vapelight.kicad_sch")
 		(attr smd)
 		(fp_line
@@
 		(property ki_fp_filters "R_*")
 		(sheetname "Root")
-		(sheetfile "SBYD_vape.kicad_sch")
+		(sheetfile "vapelight.kicad_sch")
 		(attr smd)
 		(fp_line
@@
 		(property ki_fp_filters "C_*")
 		(sheetname "Root")
-		(sheetfile "SBYD_vape.kicad_sch")
+		(sheetfile "vapelight.kicad_sch")
 		(attr smd)
 		(fp_line
@@
 			)
 		)
-		(attr exclude_from_pos_files exclude_from_bom)
+		(attr board_only exclude_from_pos_files exclude_from_bom dnp)
 		(fp_line
 			(start 0.25 1)
@@
 		)
 		(fp_text user "KIKIT: width: 3mm"
-			(at -5.5 0 0)
+			(at -5.5 0 180)
 			(layer "Dwgs.User")
 			(effects
@@
 		(property ki_fp_filters "Choke_* *Coil* Inductor_* L_*")
 		(sheetname "Root")
-		(sheetfile "SBYD_vape.kicad_sch")
+		(sheetfile "vapelight.kicad_sch")
 		(attr smd)
 		(fp_line
@@
 		(property ki_fp_filters "R_*")
 		(sheetname "Root")
-		(sheetfile "SBYD_vape.kicad_sch")
+		(sheetfile "vapelight.kicad_sch")
 		(attr smd)
 		(fp_line
@@
 		)
 		(sheetname "Root")
-		(sheetfile "SBYD_vape.kicad_sch")
+		(sheetfile "vapelight.kicad_sch")
 		(attr smd)
 		(fp_line
@@
 		(property ki_fp_filters "R_*")
 		(sheetname "Root")
-		(sheetfile "SBYD_vape.kicad_sch")
+		(sheetfile "vapelight.kicad_sch")
 		(attr smd)
 		(fp_line
@@
 		(property ki_fp_filters "Choke_* *Coil* Inductor_* L_*")
 		(sheetname "Root")
-		(sheetfile "SBYD_vape.kicad_sch")
+		(sheetfile "vapelight.kicad_sch")
 		(attr smd)
 		(fp_line
@@
 		(property ki_fp_filters "TSOT?23*")
 		(sheetname "Root")
-		(sheetfile "SBYD_vape.kicad_sch")
+		(sheetfile "vapelight.kicad_sch")
 		(attr smd)
 		(fp_line
@@
 		(property ki_fp_filters "C_*")
 		(sheetname "Root")
-		(sheetfile "SBYD_vape.kicad_sch")
+		(sheetfile "vapelight.kicad_sch")
 		(attr smd)
 		(fp_line
@@
 		(property ki_fp_filters "C_*")
 		(sheetname "Root")
-		(sheetfile "SBYD_vape.kicad_sch")
+		(sheetfile "vapelight.kicad_sch")
 		(attr smd)
 		(fp_line
@@
 			)
 		)
-		(attr exclude_from_pos_files exclude_from_bom)
+		(attr board_only exclude_from_pos_files exclude_from_bom dnp)
 		(fp_line
 			(start 0.25 0)
@@
 			)
 		)
-		(property "LCSC" "C571338"
+		(property "LCSC" "C318886"
 			(at 0 0 -90)
 			(unlocked yes)
@@
 		)
 		(sheetname "Root")
-		(sheetfile "SBYD_vape.kicad_sch")
+		(sheetfile "vapelight.kicad_sch")
 		(attr smd)
 		(fp_line
@@
 		(property ki_fp_filters "SOT?23*")
 		(sheetname "Root")
-		(sheetfile "SBYD_vape.kicad_sch")
+		(sheetfile "vapelight.kicad_sch")
 		(attr smd)
 		(fp_line
@@
 		(property ki_fp_filters "TO-???* *_Diode_* *SingleDiode* D_*")
 		(sheetname "Root")
-		(sheetfile "SBYD_vape.kicad_sch")
+		(sheetfile "vapelight.kicad_sch")
 		(attr smd)
 		(fp_line
@@
 			)
 		)
+		(property ki_fp_filters "USB*")
+		(sheetname "Root")
+		(sheetfile "vapelight.kicad_sch")
 		(attr smd exclude_from_pos_files exclude_from_bom)
 		(fp_text user "${REFERENCE}"
@@
 		(property ki_fp_filters "TO-???* *_Diode_* *SingleDiode* D_*")
 		(sheetname "Root")
-		(sheetfile "SBYD_vape.kicad_sch")
+		(sheetfile "vapelight.kicad_sch")
 		(attr smd)
 		(fp_line
@@
 		(property ki_fp_filters "C_*")
 		(sheetname "Root")
-		(sheetfile "SBYD_vape.kicad_sch")
+		(sheetfile "vapelight.kicad_sch")
 		(attr smd)
 		(fp_line
@@
 		(property ki_fp_filters "SG-* SOT*")
 		(sheetname "Root")
-		(sheetfile "SBYD_vape.kicad_sch")
+		(sheetfile "vapelight.kicad_sch")
 		(attr smd)
 		(fp_line
@@
 		)
 	)
-	(gr_text "Rev.E  03/2025\nCERN OHL P 2.0\nhttps://\n  github.com/\n    sbyd-space/\n      vape-light"
+	(gr_text "Rev.${REVISION}  ${ISSUE_DATE}\nCERN OHL P 2.0\nhttps://\n  github.com/\n    sbyd-space/\n      vape-light"
 		(at 70.5 62 180)
 		(layer "B.SilkS")
@@
 	)
 	(gr_text "PCB3D_BR_vape"
-		(at 125.5 74 0)
+		(at 128 74 0)
 		(layer "User.1")
 		(effects
